Commit message: urdf fixed - origin of joints and typo in origin of links

File: robot_des.urdf (robot description, URDF)
Before this commit: robot navvis, 5 links, 4 joints
Joints:
- joint base_laser_horiz_joint: origin xyz=0.2325 0.0001 1.9201 rpy=-0.0012 0.1146 -0.0015 -> xyz=0 0 0
- joint base_laser_vert_bottom_joint: origin xyz=0.3158 -0.0021 0.5100 rpy=3.1355 -1.3045 0.0025 -> xyz=0 0 0
- joint base_laser_vert_top_left_joint: origin xyz=0.2997 0.1531 0.18451 rpy=1.1780 0.6198 1.9560 -> xyz=0 0 0
- joint base_laser_vert_top_right_joint: origin xyz=0.2978 -0.1450 1.8451 rpy=-1.1760 0.6313 -1.9377 -> xyz=0 0 0
